File: hw/kicad/v5.0/hv_drive.kicad_sch (KiCad schematic)
At the start: 28 parts, among them P6 CONN_01X02, P8 CONN_01X03, U12 IKCM30F60GAXKMA1

Commit message: Fix shunt resistor value
Parts:
- R80, R81, R82: value 0.002 -> 0.003
Changed lines of the file:
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@@
 			)
 		)
-		(property "Value" "0.002"
+		(property "Value" "0.003"
 			(at 165.1 100.33 90)
 			(effects
@@
 			)
 		)
-		(property "Value" "0.002"
+		(property "Value" "0.003"
 			(at 165.1 95.25 90)
 			(effects
@@
 			)
 		)
-		(property "Value" "0.002"
+		(property "Value" "0.003"
 			(at 165.1 90.17 90)
 			(effects
