File: hw/kicad/v5.0/hv_drive.kicad_sch (KiCad schematic)
At the start: 28 parts, among them P6 CONN_01X02, P8 CONN_01X03, U12 IKCM30F60GAXKMA1

Commit message: hw: name the fitted IKCM30F60GD instead of the GA
The v5.0 boards carry the DCB IKCM30F60GD; the KiCad files named the
fullpack IKCM30F60GA. Both datasheets (v2.5 GD, v2.7 GA, package outline
p. 15) give the same 36 x 21 mm body and lead pattern, so no copper
moves; only the heatsink notch differs (3.2 vs 3.5 mm), off the PCB.

- stmbl.kicad_sym: symbol IKCM30F60GDXKMA1, footprint, datasheet link,
  DigiKey IKCM30F60GDXKMA1-ND, Mouser 726-IKCM30F60GDXKMA1
- hv_drive.kicad_sch: U12 moves from the stmbl_4.0-rescue copy to
  stmbl:IKCM30F60GDXKMA1 (same 24 pins), same fields
- stmbl_5.0.kicad_pcb: U12 footprint name, fields and 3D model path
- footprint IKCM30F60GAXKMA1_2 -> IKCM30F60GDXKMA1, STEP model renamed;
  the four unused variants (plain, _1, the two MFG ones) removed
- doc: GD datasheet v2.5 replaces the GA v2.7
- board STEP export: product name

The interactive BOM (bom/ibom.html) stores its data compressed and needs
regenerating in KiCad.

Co-Authored-By: Claude Opus 5.5 <noreply@anthropic.com>
Claude-Session: https://claude.ai/code/session_01M9zC28zjyMcc7fQ9NSQgeV
Parts:
- U12: value IKCM30F60GAXKMA1 -> IKCM30F60GDXKMA1; footprint stmbl:IKCM30F60GAXKMA1_2 -> stmbl:IKCM30F60GDXKMA1; symbol stmbl_4.0-rescue:IKCM30F60GAXKMA1-stmbl -> stmbl:IKCM30F60GDXKMA1; digikey part number IKCM30F60GAXKMA1-ND -> IKCM30F60GDXKMA1-ND; mouser part number 726-IKCM30F60GAXKMA1 -> 726-IKCM30F60GDXKMA1
Changed lines of the file:
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@@
 	)
 	(symbol
-		(lib_id "stmbl_4.0-rescue:IKCM30F60GAXKMA1-stmbl")
+		(lib_id "stmbl:IKCM30F60GDXKMA1")
 		(at 119.38 67.31 0)
 		(unit 1)
@@
 			)
 		)
-		(property "Value" "IKCM30F60GAXKMA1"
+		(property "Value" "IKCM30F60GDXKMA1"
 			(at 137.16 60.6044 0)
 			(effects
@@
 			)
 		)
-		(property "Footprint" "stmbl:IKCM30F60GAXKMA1_2"
+		(property "Footprint" "stmbl:IKCM30F60GDXKMA1"
 			(at 137.16 62.9158 0)
 			(effects
@@
 			)
 		)
-		(property "Datasheet" "https://www.infineon.com/dgdl/Infineon-IKCM30F60GA-DS-v02_06-EN.pdf?fileId=5546d4624fb7fef2014fcb83cab8790a"
+		(property "Datasheet" "https://www.infineon.com/cms/en/product/power/intelligent-power-modules-ipm/ikcm30f60gd/"
 			(at 119.38 54.61 0)
 			(effects
@@
 			)
 		)
-		(property "digikey part number" "IKCM30F60GAXKMA1-ND"
+		(property "digikey part number" "IKCM30F60GDXKMA1-ND"
 			(at 119.38 36.83 0)
 			(effects
@@
 			)
 		)
-		(property "mouser part number" "726-IKCM30F60GAXKMA1"
+		(property "mouser part number" "726-IKCM30F60GDXKMA1"
 			(at 119.38 16.51 0)
 			(effects
