File: hw/kicad/v5.0/hv_drive.kicad_sch (KiCad schematic)
At the start: 28 parts, among them P6 CONN_01X02, P8 CONN_01X03, U12 IKCM30F60GAXKMA1

Commit message: hw v5.0: shunt value, the fitted IKCM30F60GD named, interactive BOM regenerated
- The shunts are 3 mOhm.
- The KiCad files named the fullpack IKCM30F60GA; the boards carry the DCB
  IKCM30F60GD (same body and lead pattern, only the heatsink notch
  differs): symbol, footprint, 3D model, datasheet, ERC/DRC parity.
- bom/ibom.html regenerated (KiCad 8.0.9, InteractiveHtmlBom 2.12.0):
  U12 and the 3 mOhm shunts now read right.


Co-Authored-By: Claude Opus 5.5 (1M context) <noreply@anthropic.com>
Claude-Session: https://claude.ai/code/session_01PfGZ1xgwtcbjz7i4kBXxic
Parts:
- R80, R81, R82: value 0.002 -> 0.003
- U12: value IKCM30F60GAXKMA1 -> IKCM30F60GDXKMA1; footprint stmbl:IKCM30F60GAXKMA1_2 -> stmbl:IKCM30F60GDXKMA1; symbol stmbl_4.0-rescue:IKCM30F60GAXKMA1-stmbl -> stmbl:IKCM30F60GDXKMA1; digikey part number IKCM30F60GAXKMA1-ND -> IKCM30F60GDXKMA1-ND; mouser part number 726-IKCM30F60GAXKMA1 -> 726-IKCM30F60GDXKMA1
Changed lines of the file:
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@@
 			)
 		)
-		(property "Value" "0.002"
+		(property "Value" "0.003"
 			(at 165.1 100.33 90)
 			(effects
@@
 			)
 		)
-		(property "Value" "0.002"
+		(property "Value" "0.003"
 			(at 165.1 95.25 90)
 			(effects
@@
 			)
 		)
-		(property "Value" "0.002"
+		(property "Value" "0.003"
 			(at 165.1 90.17 90)
 			(effects
@@
 	)
 	(symbol
-		(lib_id "stmbl_4.0-rescue:IKCM30F60GAXKMA1-stmbl")
+		(lib_id "stmbl:IKCM30F60GDXKMA1")
 		(at 119.38 67.31 0)
 		(unit 1)
@@
 			)
 		)
-		(property "Value" "IKCM30F60GAXKMA1"
+		(property "Value" "IKCM30F60GDXKMA1"
 			(at 137.16 60.6044 0)
 			(effects
@@
 			)
 		)
-		(property "Footprint" "stmbl:IKCM30F60GAXKMA1_2"
+		(property "Footprint" "stmbl:IKCM30F60GDXKMA1"
 			(at 137.16 62.9158 0)
 			(effects
@@
 			)
 		)
-		(property "Datasheet" "https://www.infineon.com/dgdl/Infineon-IKCM30F60GA-DS-v02_06-EN.pdf?fileId=5546d4624fb7fef2014fcb83cab8790a"
+		(property "Datasheet" "https://www.infineon.com/cms/en/product/power/intelligent-power-modules-ipm/ikcm30f60gd/"
 			(at 119.38 54.61 0)
 			(effects
@@
 			)
 		)
-		(property "digikey part number" "IKCM30F60GAXKMA1-ND"
+		(property "digikey part number" "IKCM30F60GDXKMA1-ND"
 			(at 119.38 36.83 0)
 			(effects
@@
 			)
 		)
-		(property "mouser part number" "726-IKCM30F60GAXKMA1"
+		(property "mouser part number" "726-IKCM30F60GDXKMA1"
 			(at 119.38 16.51 0)
 			(effects
