File: hw/kicad/v5.0/stmbl_5.0.kicad_pcb (KiCad board)
At the start: 2 copper layers, 99.8 x 99.8 mm, 432 parts, among them J1 RJ45_LED, J2 RJ45_LED, J3 RJ45_LED, P1 USB_C_Receptacle_USB2.0, P10 CONN_02X06, P11 USB_C_Receptacle_USB2.0, P12 CONN_01X04, P15 CONN_01X02, P2 CONN_01X02, P3 CONN_01X02, P4 CONN_01X02, P5 CONN_01X06, P6 CONN_01X02, P7 CONN_01X04, P8 CONN_01X03, P9 CONN_01X06, Q1 IRLML6344, Q2 IRLML6344, Q3 IRLML6344, Q4 IRLML6344, Q5 IRLML6344, T1 testpoint, T2 testpoint, T44 testpoint, T45 testpoint, T46 testpoint, U1 USBLC6-4SC6, U10 SN65176B, U11 SN65176B, U12 IKCM30F60GAXKMA1, U13 RT8259, U14 SN65176B, U15 SN65176B, U16 SN65176B, U17 SN65176B, U18 SN65176B, U19 SN65176B, U2 zldo1117, U20 USBLC6-4SC6, U21 USBLC6-4SC6, U22 USBLC6-4SC6, U23 USBLC6-4SC6, U234 fan, U24 RT8259, U25 STM32F303CBTx, U26 STM32F405VG, U28 RT8259, U29 USBLC6-4SC6, U3 SI8621, U4 RT8259, U5 LNK304D, U6 LM358, U7 LM358, U8 SN65176B, U9 SN65176B, Y1 8M, Y2 8M

Commit message: Fix shunt resistor value
Parts:
- R80, R81, R82: value 0.002 -> 0.003
Changed lines of the file:
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@@
 			)
 		)
-		(property "Value" "0.002"
+		(property "Value" "0.003"
 			(at 0 2.6 0)
 			(layer "F.Fab")
@@
 			)
 		)
-		(property "Value" "0.002"
+		(property "Value" "0.003"
 			(at 0 2.6 0)
 			(layer "F.Fab")
@@
 			)
 		)
-		(property "Value" "0.002"
+		(property "Value" "0.003"
 			(at 0 2.6 0)
 			(layer "F.Fab")
