File: hw/kicad/v5.0/stmbl_5.0.kicad_pcb (KiCad board)
At the start: 2 copper layers, 99.8 x 99.8 mm, 432 parts, among them J1 RJ45_LED, J2 RJ45_LED, J3 RJ45_LED, P1 USB_C_Receptacle_USB2.0, P10 CONN_02X06, P11 USB_C_Receptacle_USB2.0, P12 CONN_01X04, P15 CONN_01X02, P2 CONN_01X02, P3 CONN_01X02, P4 CONN_01X02, P5 CONN_01X06, P6 CONN_01X02, P7 CONN_01X04, P8 CONN_01X03, P9 CONN_01X06, Q1 IRLML6344, Q2 IRLML6344, Q3 IRLML6344, Q4 IRLML6344, Q5 IRLML6344, T1 testpoint, T2 testpoint, T44 testpoint, T45 testpoint, T46 testpoint, U1 USBLC6-4SC6, U10 SN65176B, U11 SN65176B, U12 IKCM30F60GAXKMA1, U13 RT8259, U14 SN65176B, U15 SN65176B, U16 SN65176B, U17 SN65176B, U18 SN65176B, U19 SN65176B, U2 zldo1117, U20 USBLC6-4SC6, U21 USBLC6-4SC6, U22 USBLC6-4SC6, U23 USBLC6-4SC6, U234 fan, U24 RT8259, U25 STM32F303CBTx, U26 STM32F405VG, U28 RT8259, U29 USBLC6-4SC6, U3 SI8621, U4 RT8259, U5 LNK304D, U6 LM358, U7 LM358, U8 SN65176B, U9 SN65176B, Y1 8M, Y2 8M

Commit message: hw: name the fitted IKCM30F60GD instead of the GA
The v5.0 boards carry the DCB IKCM30F60GD; the KiCad files named the
fullpack IKCM30F60GA. Both datasheets (v2.5 GD, v2.7 GA, package outline
p. 15) give the same 36 x 21 mm body and lead pattern, so no copper
moves; only the heatsink notch differs (3.2 vs 3.5 mm), off the PCB.

- stmbl.kicad_sym: symbol IKCM30F60GDXKMA1, footprint, datasheet link,
  DigiKey IKCM30F60GDXKMA1-ND, Mouser 726-IKCM30F60GDXKMA1
- hv_drive.kicad_sch: U12 moves from the stmbl_4.0-rescue copy to
  stmbl:IKCM30F60GDXKMA1 (same 24 pins), same fields
- stmbl_5.0.kicad_pcb: U12 footprint name, fields and 3D model path
- footprint IKCM30F60GAXKMA1_2 -> IKCM30F60GDXKMA1, STEP model renamed;
  the four unused variants (plain, _1, the two MFG ones) removed
- doc: GD datasheet v2.5 replaces the GA v2.7
- board STEP export: product name

The interactive BOM (bom/ibom.html) stores its data compressed and needs
regenerating in KiCad.

Co-Authored-By: Claude Opus 5.5 <noreply@anthropic.com>
Claude-Session: https://claude.ai/code/session_01M9zC28zjyMcc7fQ9NSQgeV
Parts:
- U12: value IKCM30F60GAXKMA1 -> IKCM30F60GDXKMA1; footprint stmbl:IKCM30F60GAXKMA1_2 -> stmbl:IKCM30F60GDXKMA1
Changed lines of the file:
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@@
 		)
 	)
-	(footprint "stmbl:IKCM30F60GAXKMA1_2"
+	(footprint "stmbl:IKCM30F60GDXKMA1"
 		(layer "B.Cu")
 		(at 154.126031 138.888474 -90)
@@
 			)
 		)
-		(property "Value" "IKCM30F60GAXKMA1"
+		(property "Value" "IKCM30F60GDXKMA1"
 			(at -14.7 14.3 90)
 			(layer "B.SilkS")
@@
 			)
 		)
-		(property "Footprint" "stmbl:IKCM30F60GAXKMA1_2"
+		(property "Footprint" "stmbl:IKCM30F60GDXKMA1"
 			(at 0 0 -90)
 			(unlocked yes)
@@
 			)
 		)
-		(property "Datasheet" "https://www.infineon.com/dgdl/Infineon-IKCM30F60GA-DS-v02_06-EN.pdf?fileId=5546d4624fb7fef2014fcb83cab8790a"
+		(property "Datasheet" "https://www.infineon.com/cms/en/product/power/intelligent-power-modules-ipm/ikcm30f60gd/"
 			(at 0 0 -90)
 			(unlocked yes)
@@
 			)
 		)
-		(property "digikey part number" "IKCM30F60GAXKMA1-ND"
+		(property "digikey part number" "IKCM30F60GDXKMA1-ND"
 			(at 0 0 0)
 			(layer "B.Fab")
@@
 			)
 		)
-		(property "mouser part number" "726-IKCM30F60GAXKMA1"
+		(property "mouser part number" "726-IKCM30F60GDXKMA1"
 			(at 0 0 0)
 			(layer "B.Fab")
@@
 			(pintype "passive")
 		)
-		(model "${STMBL}/stmbl.pretty/Infineon_-_IKCM30F60GAXKMA1.step"
+		(model "${STMBL}/stmbl.pretty/Infineon_-_IKCM30F60GDXKMA1.step"
 			(offset
 				(xyz -15.1 16 0.2)
